File: electronics/TurntableStrobe.sch (EAGLE design)
At the start: 16 parts, among them IC1 TINY25, J1 ISP, Q1 12MHz

Commit message: added solder jumper for easier reprogramming. Minor silk tweaks. New logo.
Parts:
- added JP1: pgm, SparkFun-Retired:JUMPER-2SMD-NO
- added U$5: BTLOGO-LOGO-MD, bt:BTLOGO-LOGO-MD
Connections:
- new net N$1: JP1.2, R3.2
- net PB0: now also JP1.1; no longer R3.2
Other:
- note added: "R0.3"
- note added: "TURNTABLE STROBE"
- note added: "to program, unsolder pgm jumper"
- note removed: "R0.2"
- note removed: "Turntable Strobe"
- moved on the sheet: C1, C2, C3, C4, C5, CR1225, D1, D2, IC1, J1, LED1, Q1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
