File: electronics/handheld/TurntableStrobe.brd (EAGLE design)
At the start: 25.1 x 17.8 mm, 17 parts, among them J1 ISP, Q1 12MHz, Q2 BJT-NPNSOT23, U1 TINY25, U2 LM2665

Commit message: updated supply caps
Parts:
- C2: value 10uF -> 47uF
Changed lines of the file:
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@@
 <attribute name="NAME" x="13.97" y="13.081" size="0.8128" layer="25" font="vector" ratio="10" rot="R180"/>
 </element>
-<element name="C2" library="rcl" package="C0603" value="10uF" x="2.54" y="15.367" smashed="yes" rot="R270">
+<element name="C2" library="rcl" package="C0603" value="47uF" x="2.54" y="15.367" smashed="yes" rot="R270">
 <attribute name="NAME" x="2.667" y="13.335" size="0.8128" layer="25" font="vector" ratio="10" rot="R180" align="center"/>
 </element>
